File: ArduinoShield.kicad_pcb (KiCad board)
At the start: 2 copper layers, 19 parts, among them J1 pulX, J2 dirX, J3 enaX, J4 pulY, J5 dirY, J6 enaY, J7 pulZ, J8 dirZ, J9 enaZ, Q1 Q_NPN_CBE, Q2 Q_NPN_CBE, Q3 Q_NPN_CBE, Q4 Q_NPN_CBE, Q5 Q_NPN_CBE, Q6 Q_NPN_CBE, Q7 Q_NPN_CBE, Q8 Q_NPN_CBE, Q9 Q_NPN_CBE

Commit message: Add files via upload
Parts:
- added Q10: PN2222A, TO_SOT_Packages_THT:TO-92_Molded_Narrow, F.Cu at (47.6, 19.7)
- added Q11: PN2222A, TO_SOT_Packages_THT:TO-92_Molded_Narrow, F.Cu at (29.8, 1.91)
- added Q12: PN2222A, TO_SOT_Packages_THT:TO-92_Molded_Narrow, F.Cu at (22.2, -5.71)
- added Q13: PN2222A, TO_SOT_Packages_THT:TO-92_Molded_Narrow, F.Cu at (13.3, -5.71)
- added U1: NE555, Housings_DIP:DIP-8_W7.62mm_Socket_LongPads, F.Cu at (22.2, 32.4)
Connections:
- net Net-(XA1-PadA0) renamed /force/forceOut

Commit message: Add files via upload
Parts:
- added C1: C, Capacitors_THT:C_Disc_D6.0mm_W2.5mm_P5.00mm, F.Cu at (25.7, 144.2)
- added C2: CP, Capacitors_THT:CP_Radial_D4.0mm_P1.50mm, F.Cu at (47.4, 101.2)
- added C3: CP, Capacitors_THT:CP_Radial_D5.0mm_P2.00mm, F.Cu at (59.3, 93.2)
- added D1: D, Diodes_THT:D_DO-35_SOD27_P7.62mm_Horizontal, F.Cu at (75.9, 153.4)
- added D2: D, Diodes_THT:D_DO-35_SOD27_P7.62mm_Horizontal, F.Cu at (75.9, 141.5)
- added J10: Flex_Sensor, Connectors_Terminal_Blocks:TerminalBlock_Altech_AK300-2_P5.00mm, F.Cu at (101.7, 147.4)
- added J11: VFD analog Voltage, Connectors_Terminal_Blocks:TerminalBlock_Altech_AK300-2_P5.00mm, F.Cu at (273.8, 124.4)
- added J12: Forward/Stop, Connectors_Terminal_Blocks:TerminalBlock_Altech_AK300-2_P5.00mm, F.Cu at (274.7, 67.0)
- added J13: Jog, Connectors_Terminal_Blocks:TerminalBlock_Altech_AK300-2_P5.00mm, F.Cu at (274.4, 110.7)
- added J14: External Faul(N 0), Connectors_Terminal_Blocks:TerminalBlock_Altech_AK300-2_P5.00mm, F.Cu at (274.0, 97.1)
- added J15: Reverse/Stop, Connectors_Terminal_Blocks:TerminalBlock_Altech_AK300-2_P5.00mm, F.Cu at (274.5, 81.4)
- added J16: pulX0, Connectors_Terminal_Blocks:TerminalBlock_Altech_AK300-2_P5.00mm, F.Cu at (127.2, 23.5)
- added J17: dirX0, Connectors_Terminal_Blocks:TerminalBlock_Altech_AK300-2_P5.00mm, F.Cu at (140.2, 23.5)
- added J18: enaX0, Connectors_Terminal_Blocks:TerminalBlock_Altech_AK300-2_P5.00mm, F.Cu at (153.2, 23.5)
- added J19: MAX6675, Socket_Strips:Socket_Strip_Straight_1x05_Pitch2.54mm, F.Cu at (240.4, 76.0)
- added J20: ASC712, Socket_Strips:Socket_Strip_Straight_1x03_Pitch2.54mm, F.Cu at (173.4, 154.1)
- added J21: +12V, Connectors_Terminal_Blocks:TerminalBlock_Altech_AK300-2_P5.00mm, F.Cu at (147.7, 158.7)
- added Q14: Q_NPN_CBE, TO_SOT_Packages_THT:TO-92_Inline_Narrow_Oval, F.Cu at (127.9, 36.8)
- added Q15: Q_NPN_CBE, TO_SOT_Packages_THT:TO-92_Inline_Narrow_Oval, F.Cu at (140.1, 36.9)
- added Q16: Q_NPN_CBE, TO_SOT_Packages_THT:TO-92_Inline_Narrow_Oval, F.Cu at (153.8, 36.9)
- added R1: R, Resistors_THT:R_Axial_DIN0207_L6.3mm_D2.5mm_P10.16mm_Horizontal, F.Cu at (63.0, 126.2)
- added R10: R, Resistors_THT:R_Axial_DIN0207_L6.3mm_D2.5mm_P10.16mm_Horizontal, F.Cu at (170.9, 32.9)
- added R11: R, Resistors_THT:R_Axial_DIN0207_L6.3mm_D2.5mm_P10.16mm_Horizontal, F.Cu at (183.6, 33.1)
- added R12: R, Resistors_THT:R_Axial_DIN0207_L6.3mm_D2.5mm_P10.16mm_Horizontal, F.Cu at (196.1, 33.1)
- added R13: R, Resistors_THT:R_Axial_DIN0207_L6.3mm_D2.5mm_P10.16mm_Horizontal, F.Cu at (209.1, 33.1)
- added R14: R, Resistors_THT:R_Axial_DIN0207_L6.3mm_D2.5mm_P10.16mm_Horizontal, F.Cu at (222.1, 33.1)
- added R15: R, Resistors_THT:R_Axial_DIN0207_L6.3mm_D2.5mm_P10.16mm_Horizontal, F.Cu at (235.1, 33.1)
- added R16: R, Resistors_THT:R_Axial_DIN0207_L6.3mm_D2.5mm_P10.16mm_Horizontal, F.Cu at (248.1, 33.1)
- added R17: R, Resistors_THT:R_Axial_DIN0207_L6.3mm_D2.5mm_P10.16mm_Horizontal, F.Cu at (261.9, 33.0)
- added R18: R, Resistors_THT:R_Axial_DIN0207_L6.3mm_D2.5mm_P10.16mm_Horizontal, F.Cu at (274.1, 33.1)
- added R2: R, Resistors_THT:R_Axial_DIN0207_L6.3mm_D2.5mm_P10.16mm_Horizontal, F.Cu at (62.7, 142.0)
- added R3: R, Resistors_THT:R_Axial_DIN0207_L6.3mm_D2.5mm_P10.16mm_Horizontal, F.Cu at (73.8, 105.7)
- added R4: R, Resistors_THT:R_Axial_DIN0207_L6.3mm_D2.5mm_P10.16mm_Horizontal, F.Cu at (105.9, 122.9)
- added R5: R, Resistors_THT:R_Axial_DIN0207_L6.3mm_D2.5mm_P10.16mm_Horizontal, F.Cu at (260.2, 142.5)
- added R6: R, Resistors_THT:R_Axial_DIN0207_L6.3mm_D2.5mm_P10.16mm_Horizontal, F.Cu at (263.4, 123.2)
- added R7: R, Resistors_THT:R_Axial_DIN0207_L6.3mm_D2.5mm_P10.16mm_Horizontal, F.Cu at (132.2, 33.1)
- added R8: R, Resistors_THT:R_Axial_DIN0207_L6.3mm_D2.5mm_P10.16mm_Horizontal, F.Cu at (145.1, 33.1)
- added R9: R, Resistors_THT:R_Axial_DIN0207_L6.3mm_D2.5mm_P10.16mm_Horizontal, F.Cu at (158.3, 33.0)
- added RV1: POT, Potentiometers:Potentiometer_WirePads_largePads, F.Cu at (74.3, 90.7)
- added RV2: POT, Potentiometers:Potentiometer_WirePads_largePads, F.Cu at (128.9, 150.6)
- added U2: LM337_TO220, TO_SOT_Packages_THT:TO-220-3_Vertical, F.Cu at (56.6, 114.1)
- added U3: MCP6004, Housings_DIP:DIP-8_W10.16mm_LongPads, F.Cu at (128.7, 131.1)
- added U4: LM741, Housings_DIP:DIP-8_W10.16mm_LongPads, F.Cu at (250.8, 133.3)
- J1: value pulX -> pulX1
- J2: value dirX -> dirX1
- J3: value enaX -> enaX1
- moved Q13 270.3 mm to (257.1, 110.9)
- moved Q12 256.1 mm to (257.6, 95.2)
- moved Q11 241.6 mm to (258.1, 81.2)
- moved Q10 215.7 mm to (258.0, 67.0)
- moved U1 115.6 mm to (49.7, 144.7), turned to 180 degrees
- moved J1 3.61 mm to (165.9, 23.6)
- moved J2 3.61 mm to (178.6, 23.6)
- moved J3 3.61 mm to (191.3, 23.6)
- moved J4 3.61 mm to (204.0, 23.6)
- moved J5 3.61 mm to (216.7, 23.6)
- moved J6 3.61 mm to (230.0, 23.6)
- moved J7 3.61 mm to (243.4, 23.6)
- moved J8 3.61 mm to (256.7, 23.6)
- moved J9 3.61 mm to (269.4, 23.6)
- moved Q3 2.80 mm to (190.9, 36.9), turned to 180 degrees
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Connections:
- Q1 pad 1: Net-(J1-Pad2) -> Net-(Q1-Pad1)
- Q1 pad 2: /Stepper/PulX -> (no net)
- Q10 pad 2: /vfd/Forward/Stop -> (no net)
- Q11 pad 2: /vfd/Reverse/Stop -> (no net)
- Q12 pad 2: /vfd/externalFault -> (no net)
- Q13 pad 2: /vfd/jog -> (no net)
- Q2 pad 1: Net-(J2-Pad2) -> Net-(Q2-Pad1)
- Q2 pad 2: /Stepper/dirX -> (no net)
- Q3 pad 1: Net-(J3-Pad2) -> Net-(Q3-Pad1)
- Q3 pad 2: /Stepper/enaX -> (no net)
- Q4 pad 1: Net-(J4-Pad2) -> Net-(Q4-Pad1)
- Q5 pad 1: Net-(J5-Pad2) -> Net-(Q5-Pad1)
- Q6 pad 1: Net-(J6-Pad2) -> Net-(Q6-Pad1)
- Q7 pad 1: Net-(J7-Pad2) -> Net-(Q7-Pad1)
- Q8 pad 1: Net-(J8-Pad2) -> Net-(Q8-Pad1)
- Q9 pad 1: Net-(J9-Pad2) -> Net-(Q9-Pad1)
- XA1 pad 3V3: Net-(XA1-Pad3V3) -> (no net)
- XA1 pad 5V1: Net-(XA1-Pad5V1) -> +5V
- XA1 pad 5V2: Net-(XA1-Pad5V2) -> (no net)
- XA1 pad 5V3: Net-(XA1-Pad5V3) -> +5V
- XA1 pad 5V4: Net-(XA1-Pad5V4) -> +5V
- XA1 pad A1: Net-(XA1-PadA1) -> (no net)
- XA1 pad A10: Net-(XA1-PadA10) -> (no net)
- XA1 pad A11: Net-(XA1-PadA11) -> (no net)
- XA1 pad A12: Net-(XA1-PadA12) -> (no net)
- XA1 pad A13: Net-(XA1-PadA13) -> (no net)
- XA1 pad A14: Net-(XA1-PadA14) -> (no net)
- XA1 pad A15: Net-(XA1-PadA15) -> (no net)
- XA1 pad A2: Net-(XA1-PadA2) -> (no net)
- XA1 pad A3: Net-(XA1-PadA3) -> (no net)
- XA1 pad A4: Net-(XA1-PadA4) -> (no net)
- XA1 pad A5: Net-(XA1-PadA5) -> (no net)
- XA1 pad A6: Net-(XA1-PadA6) -> (no net)
- XA1 pad A7: Net-(XA1-PadA7) -> (no net)
- XA1 pad A8: Net-(XA1-PadA8) -> (no net)
- XA1 pad A9: Net-(XA1-PadA9) -> (no net)
- XA1 pad AREF: Net-(XA1-PadAREF) -> (no net)
- XA1 pad D0: Net-(XA1-PadD0) -> (no net)
- XA1 pad D1: Net-(XA1-PadD1) -> (no net)
- XA1 pad D11: Net-(XA1-PadD11) -> (no net)
- XA1 pad D13: /Stepper/PulX -> (no net)
- XA1 pad D14: Net-(XA1-PadD14) -> (no net)
- XA1 pad D15: Net-(XA1-PadD15) -> (no net)
- XA1 pad D16: Net-(XA1-PadD16) -> (no net)
- XA1 pad D17: Net-(XA1-PadD17) -> (no net)
- XA1 pad D18: Net-(XA1-PadD18) -> (no net)
- XA1 pad D19: Net-(XA1-PadD19) -> (no net)
- XA1 pad D2: Net-(XA1-PadD2) -> (no net)
- XA1 pad D20: Net-(XA1-PadD20) -> (no net)
- XA1 pad D21: Net-(XA1-PadD21) -> (no net)
- XA1 pad D22: /Stepper/dirX -> (no net)
- XA1 pad D23: /Stepper/enaX -> (no net)
- XA1 pad D28: Net-(XA1-PadD28) -> (no net)
- XA1 pad D29: Net-(XA1-PadD29) -> (no net)
- XA1 pad D3: Net-(XA1-PadD3) -> (no net)
- XA1 pad D30: Net-(XA1-PadD30) -> (no net)
- XA1 pad D31: Net-(XA1-PadD31) -> (no net)
- XA1 pad D32: Net-(XA1-PadD32) -> (no net)
- XA1 pad D33: Net-(XA1-PadD33) -> (no net)
- XA1 pad D34: Net-(XA1-PadD34) -> (no net)
- XA1 pad D35: Net-(XA1-PadD35) -> (no net)
- XA1 pad D36: Net-(XA1-PadD36) -> (no net)
- XA1 pad D37: Net-(XA1-PadD37) -> (no net)
- XA1 pad D38: Net-(XA1-PadD38) -> (no net)
- XA1 pad D39: Net-(XA1-PadD39) -> (no net)
- XA1 pad D4: Net-(XA1-PadD4) -> (no net)
- XA1 pad D40: Net-(XA1-PadD40) -> (no net)
- XA1 pad D41: Net-(XA1-PadD41) -> (no net)
- XA1 pad D42: Net-(XA1-PadD42) -> (no net)
- XA1 pad D43: Net-(XA1-PadD43) -> (no net)
- XA1 pad D44: Net-(XA1-PadD44) -> (no net)
- XA1 pad D45: Net-(XA1-PadD45) -> (no net)
- XA1 pad D46: Net-(XA1-PadD46) -> (no net)
- XA1 pad D47: Net-(XA1-PadD47) -> (no net)
- XA1 pad D48: Net-(XA1-PadD48) -> (no net)
- XA1 pad D49: Net-(XA1-PadD49) -> (no net)
- XA1 pad D5: Net-(XA1-PadD5) -> (no net)
- XA1 pad D50: Net-(XA1-PadD50) -> (no net)
- XA1 pad D51: Net-(XA1-PadD51) -> (no net)
- XA1 pad D52: Net-(XA1-PadD52) -> (no net)
- XA1 pad D53: Net-(XA1-PadD53) -> (no net)
- XA1 pad D6: Net-(XA1-PadD6) -> (no net)
- XA1 pad D7: Net-(XA1-PadD7) -> (no net)
- XA1 pad D8: Net-(XA1-PadD8) -> (no net)
- XA1 pad D9: Net-(XA1-PadD9) -> (no net)
- XA1 pad GND4: Net-(XA1-PadGND4) -> (no net)
- XA1 pad IORF: Net-(XA1-PadIORF) -> (no net)
- XA1 pad MISO: Net-(XA1-PadMISO) -> (no net)
- XA1 pad MOSI: Net-(XA1-PadMOSI) -> (no net)
- XA1 pad RST1: Net-(XA1-PadRST1) -> (no net)
- XA1 pad RST2: Net-(XA1-PadRST2) -> (no net)
- XA1 pad SCK: Net-(XA1-PadSCK) -> (no net)
- XA1 pad SCL: Net-(XA1-PadSCL) -> (no net)
- XA1 pad SDA: Net-(XA1-PadSDA) -> (no net)
Routing:
- net Net-(J1-Pad2): track 36.9 -> 9.29 mm
- net Net-(J16-Pad2): track 0.00 -> 9.68 mm
- net Net-(J17-Pad2): track 0.00 -> 9.60 mm
- net Net-(J18-Pad2): track 0.00 -> 9.45 mm
- net Net-(Q1-Pad1): track 0.00 -> 9.22 mm
- net Net-(J6-Pad2): track 18.5 -> 9.48 mm
- net Net-(J4-Pad2): track 18.5 -> 9.50 mm
- net Net-(J2-Pad2): track 18.5 -> 9.54 mm
- net Net-(J7-Pad2): track 18.5 -> 9.61 mm
- net Net-(J5-Pad2): track 18.5 -> 9.62 mm
- net Net-(Q2-Pad1): track 0.00 -> 8.71 mm
- net Net-(J3-Pad2): track 18.3 -> 9.58 mm
- net Net-(J8-Pad2): track 18.5 -> 10.0 mm
- net Net-(Q3-Pad1): track 0.00 -> 8.43 mm
- net Net-(Q15-Pad1): track 0.00 -> 8.34 mm
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Other:
- net class Default: clearance 0.2 -> 0.25; trace_width 0.25 -> 0.4
- rule trace_clearance: 0.2 -> 0.25

Commit message: Add files via upload
Parts:
- moved J19 85.6 mm to (211.7, 156.7), turned to 90 degrees
Changed lines of the file:
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@@
     (links 115)
     (no_connects 65)
-    (area 0 0 0 0)
+    (area 12.7 12.7 283.845001 166.81)
     (thickness 1.6)
     (drawings 1)
@@
   )
   (module Socket_Strips:Socket_Strip_Straight_1x05_Pitch2.54mm (layer F.Cu)
-    (at 240.425 76.035)
+    (at 211.725 156.665 90)
     (descr "Through hole straight socket strip, 1x05, 2.54mm pitch, single row")
     (tags "Through hole socket strip THT 1x05 2.54mm single row")
-    (fp_text reference J19 (at 0 -2.33) (layer F.SilkS)
+    (fp_text reference J19 (at 0 -2.33 90) (layer F.SilkS)
       (effects (font (size 1 1) (thickness 0.15)))
     )
-    (fp_text value MAX6675 (at 0 12.49) (layer F.Fab)
+    (fp_text value MAX6675 (at 0 12.49 90) (layer F.Fab)
       (effects (font (size 1 1) (thickness 0.15)))
     )
@@
     (fp_line (start 1.8 11.95) (end 1.8 -1.8) (layer F.CrtYd) (width 0.05))
     (fp_line (start 1.8 -1.8) (end -1.8 -1.8) (layer F.CrtYd) (width 0.05))
-    (fp_text user %R (at 0 -2.33) (layer F.Fab)
+    (fp_text user %R (at 0 -2.33 90) (layer F.Fab)
       (effects (font (size 1 1) (thickness 0.15)))
     )
-    (pad 1 thru_hole rect (at 0 0) (size 1.7 1.7) (drill 1) (layers *.Cu *.Mask)
+    (pad 1 thru_hole rect (at 0 0 90) (size 1.7 1.7) (drill 1) (layers *.Cu *.Mask)
       (net 11 GND))
-    (pad 2 thru_hole oval (at 0 2.54) (size 1.7 1.7) (drill 1) (layers *.Cu *.Mask)
+    (pad 2 thru_hole oval (at 0 2.54 90) (size 1.7 1.7) (drill 1) (layers *.Cu *.Mask)
       (net 1 +5V))
-    (pad 3 thru_hole oval (at 0 5.08) (size 1.7 1.7) (drill 1) (layers *.Cu *.Mask))
-    (pad 4 thru_hole oval (at 0 7.62) (size 1.7 1.7) (drill 1) (layers *.Cu *.Mask))
-    (pad 5 thru_hole oval (at 0 10.16) (size 1.7 1.7) (drill 1) (layers *.Cu *.Mask))
+    (pad 3 thru_hole oval (at 0 5.08 90) (size 1.7 1.7) (drill 1) (layers *.Cu *.Mask))
+    (pad 4 thru_hole oval (at 0 7.62 90) (size 1.7 1.7) (drill 1) (layers *.Cu *.Mask))
+    (pad 5 thru_hole oval (at 0 10.16 90) (size 1.7 1.7) (drill 1) (layers *.Cu *.Mask))
     (model ${KISYS3DMOD}/Socket_Strips.3dshapes/Socket_Strip_Straight_1x05_Pitch2.54mm.wrl
       (at (xyz 0 -0.2 0))

Commit message: Add files via upload
Parts:
- moved Q13 0.95 mm to (258.1, 110.9)
- moved Q12 0.45 mm to (258.1, 95.2)
- moved Q10 0.23 mm to (258.3, 66.9)
Changed lines of the file:
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@@
   (general
     (links 115)
-    (no_connects 65)
+    (no_connects 64)
     (area 12.7 12.7 283.845001 166.81)
     (thickness 1.6)
@@
       (effects (font (size 1 1) (thickness 0.15)))
     )
-    (fp_text value dirX0 (at 5.842 -7.366 180) (layer F.Fab)
+    (fp_text value dirX0 (at 5.842 -7.366) (layer F.SilkS)
       (effects (font (size 1 1) (thickness 0.15)))
     )
@@
       (effects (font (size 1 1) (thickness 0.15)))
     )
-    (fp_text value Arduino_Mega2560_Shield (at 15.494 -54.356) (layer F.Fab)
+    (fp_text value Arduino_Mega2560_Shield (at 15.494 -54.356) (layer F.SilkS)
       (effects (font (size 1 1) (thickness 0.15)))
     )
@@
       (effects (font (size 1 1) (thickness 0.15)))
     )
-    (fp_text value pulX1 (at 5.461 -7.493) (layer F.Fab)
+    (fp_text value pulX1 (at 5.461 -7.493) (layer F.SilkS)
       (effects (font (size 1 1) (thickness 0.15)))
     )
@@
       (effects (font (size 1 1) (thickness 0.15)))
     )
-    (fp_text value dirX1 (at 5.455 -7.525) (layer F.Fab)
+    (fp_text value dirX1 (at 5.455 -7.525) (layer F.SilkS)
       (effects (font (size 1 1) (thickness 0.15)))
     )
@@
       (effects (font (size 1 1) (thickness 0.15)))
     )
-    (fp_text value enaX1 (at 5.755 -7.525 180) (layer F.Fab)
+    (fp_text value enaX1 (at 5.755 -7.525) (layer F.SilkS)
       (effects (font (size 1 1) (thickness 0.15)))
     )
@@
       (effects (font (size 1 1) (thickness 0.15)))
     )
-    (fp_text value pulY (at 6.055 -7.525) (layer F.Fab)
+    (fp_text value pulY (at 6.055 -7.525) (layer F.SilkS)
       (effects (font (size 1 1) (thickness 0.15)))
     )
@@
       (effects (font (size 1 1) (thickness 0.15)))
     )
-    (fp_text value dirY (at 5.795 -7.435) (layer F.Fab)
+    (fp_text value dirY (at 5.795 -7.435) (layer F.SilkS)
       (effects (font (size 1 1) (thickness 0.15)))
     )
@@
       (effects (font (size 1 1) (thickness 0.15)))
     )
-    (fp_text value enaY (at 5.72 -7.585) (layer F.Fab)
+    (fp_text value enaY (at 5.72 -7.585) (layer F.SilkS)
       (effects (font (size 1 1) (thickness 0.15)))
     )
@@
       (effects (font (size 1 1) (thickness 0.15)))
     )
-    (fp_text value pulZ (at 5.585 -7.555) (layer F.Fab)
+    (fp_text value pulZ (at 5.585 -7.555) (layer F.SilkS)
       (effects (font (size 1 1) (thickness 0.15)))
     )
@@
       (effects (font (size 1 1) (thickness 0.15)))
     )
-    (fp_text value dirZ (at 5.05 -7.665) (layer F.Fab)
+    (fp_text value dirZ (at 5.05 -7.665) (layer F.SilkS)
       (effects (font (size 1 1) (thickness 0.15)))
     )
@@
       (effects (font (size 1 1) (thickness 0.15)))
     )
-    (fp_text value enaZ (at 5.31 -7.995) (layer F.Fab)
+    (fp_text value enaZ (at 2.47 -7.945) (layer F.SilkS)
       (effects (font (size 1 1) (thickness 0.15)))
     )
@@
   )
   (module TO_SOT_Packages_THT:TO-92_Molded_Narrow (layer F.Cu)
-    (at 258.025 66.985)
+    (at 258.255 66.945)
     (descr "TO-92 leads molded, narrow, drill 0.6mm (see NXP sot054_po.pdf)")
     (tags "to-92 sc-43 sc-43a sot54 PA33 transistor")
@@
   )
   (module TO_SOT_Packages_THT:TO-92_Molded_Narrow (layer F.Cu)
-    (at 258.085 81.175)
+    (at 258.075 81.165)
     (descr "TO-92 leads molded, narrow, drill 0.6mm (see NXP sot054_po.pdf)")
     (tags "to-92 sc-43 sc-43a sot54 PA33 transistor")
@@
   )
   (module TO_SOT_Packages_THT:TO-92_Molded_Narrow (layer F.Cu)
-    (at 257.635 95.195)
+    (at 258.085 95.215)
     (descr "TO-92 leads molded, narrow, drill 0.6mm (see NXP sot054_po.pdf)")
     (tags "to-92 sc-43 sc-43a sot54 PA33 transistor")
@@
   )
   (module TO_SOT_Packages_THT:TO-92_Molded_Narrow (layer F.Cu)
-    (at 257.135 110.905)
+    (at 258.085 110.905)
     (descr "TO-92 leads molded, narrow, drill 0.6mm (see NXP sot054_po.pdf)")
     (tags "to-92 sc-43 sc-43a sot54 PA33 transistor")
@@
       (effects (font (size 1 1) (thickness 0.15)))
     )
-    (fp_text value Flex_Sensor (at 2.78 7.75 180) (layer F.Fab)
+    (fp_text value Flex_Sensor (at 2.78 7.75 180) (layer F.SilkS)
       (effects (font (size 1 1) (thickness 0.15)))
     )
@@
       (effects (font (size 1 1) (thickness 0.15)))
     )
-    (fp_text value "VFD analog Voltage" (at 2.78 7.75 270) (layer F.Fab)
+    (fp_text value "VFD analog Voltage" (at 2.78 7.75 270) (layer F.SilkS)
       (effects (font (size 1 1) (thickness 0.15)))
     )
@@
       (effects (font (size 1 1) (thickness 0.15)))
     )
-    (fp_text value Forward/Stop (at 2.78 7.75 270) (layer F.Fab)
+    (fp_text value Forward/Stop (at 2.78 7.75 270) (layer F.SilkS)
       (effects (font (size 1 1) (thickness 0.15)))
     )
-    (fp_text user %R (at 1.14 -6.61 270) (layer F.Fab)
+    (fp_text user %R (at 2.68 -1.75 270) (layer F.Fab)
       (effects (font (size 1 1) (thickness 0.15)))
     )
@@
       (effects (font (size 1 1) (thickness 0.15)))
     )
-    (fp_text value Jog (at 2.78 7.75 270) (layer F.Fab)
+    (fp_text value Jog (at 2.78 7.75 270) (layer F.SilkS)
       (effects (font (size 1 1) (thickness 0.15)))
     )
@@
       (effects (font (size 1 1) (thickness 0.15)))
     )
-    (fp_text value "External Faul(N 0)" (at 2.78 7.75 270) (layer F.Fab)
+    (fp_text value "External Faul(N 0)" (at 2.78 7.75 270) (layer F.SilkS)
       (effects (font (size 1 1) (thickness 0.15)))
     )
@@
       (effects (font (size 1 1) (thickness 0.15)))
     )
-    (fp_text value Reverse/Stop (at 2.78 7.75 270) (layer F.Fab)
+    (fp_text value Reverse/Stop (at 2.78 7.75 270) (layer F.SilkS)
       (effects (font (size 1 1) (thickness 0.15)))
     )
@@
       (effects (font (size 1 1) (thickness 0.15)))
     )
-    (fp_text value pulX0 (at 5.588 -7.62) (layer F.Fab)
+    (fp_text value pulX0 (at 5.588 -7.62) (layer F.SilkS)
       (effects (font (size 1 1) (thickness 0.15)))
     )
@@
       (effects (font (size 1 1) (thickness 0.15)))
     )
-    (fp_text value enaX0 (at 6.096 -7.366) (layer F.Fab)
+    (fp_text value enaX0 (at 6.096 -7.366) (layer F.SilkS)
       (effects (font (size 1 1) (thickness 0.15)))
     )
@@
       (effects (font (size 1 1) (thickness 0.15)))
     )
-    (fp_text value MAX6675 (at 0 12.49 90) (layer F.Fab)
+    (fp_text value MAX6675 (at 0 12.49 90) (layer F.SilkS)
       (effects (font (size 1 1) (thickness 0.15)))
     )
@@
       (effects (font (size 1 1) (thickness 0.15)))
     )
-    (fp_text value ASC712 (at 0 7.41 90) (layer F.Fab)
+    (fp_text value ASC712 (at 0 7.41 90) (layer F.SilkS)
       (effects (font (size 1 1) (thickness 0.15)))
     )
@@
       (effects (font (size 1 1) (thickness 0.15)))
     )
-    (fp_text value +12V (at 2.78 7.75 180) (layer F.Fab)
+    (fp_text value +12V (at 2.78 7.75 180) (layer F.SilkS)
       (effects (font (size 1 1) (thickness 0.15)))
     )
@@
     )
   )
-  (gr_text "2017-18 Rascal PCB V1\n" (at 30.225 158.915 180) (layer F.SilkS)
+  (gr_text "2017-18 Rascal PCB V1\n" (at 28.955 159.765) (layer F.SilkS)
     (effects (font (size 1.5 1.5) (thickness 0.3)))
   )

Commit message: Add files via upload
Parts:
- added J22: xMin, Connectors_Terminal_Blocks:TerminalBlock_Altech_AK300-2_P5.00mm, F.Cu at (220.5, 150.9)
- added J23: xMax, Connectors_Terminal_Blocks:TerminalBlock_Altech_AK300-2_P5.00mm, F.Cu at (234.7, 150.8)
- added J25: zMax, Connectors_Terminal_Blocks:TerminalBlock_Altech_AK300-2_P5.00mm, F.Cu at (248.4, 150.8)
- added J26: yMin, Connectors_Terminal_Blocks:TerminalBlock_Altech_AK300-2_P5.00mm, F.Cu at (261.7, 150.8)
- added J27: yMax, Connectors_Terminal_Blocks:TerminalBlock_Altech_AK300-2_P5.00mm, F.Cu at (275.3, 151.0)
- added j24: zMin, Connectors_Terminal_Blocks:TerminalBlock_Altech_AK300-2_P5.00mm, F.Cu at (206.3, 150.8)
- moved J19 125.7 mm to (120.5, 70.3), turned to 180 degrees
- moved J20 81.6 mm to (118.6, 93.7), turned to 180 degrees
- moved J10 40.1 mm to (120.0, 111.8), turned to 90 degrees
- moved XA1 38.4 mm to (138.3, 106.9)
- moved U3 26.3 mm to (103.7, 122.8)
- moved R4 26.3 mm to (80.9, 114.5)
- moved RV2 26.3 mm to (103.9, 142.3)
- moved J21 23.5 mm to (170.4, 152.6)
- moved RV1 14.0 mm to (65.2, 80.1)
- moved R5 12.0 mm to (259.4, 130.5)
- moved C1 11.7 mm to (18.4, 135.1)
- moved C2 11.7 mm to (40.1, 92.0)
- moved C3 11.7 mm to (52.0, 84.0)
- moved R3 11.7 mm to (66.5, 96.6)
- moved U2 11.7 mm to (49.3, 105.0)
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Connections:
- Q4 pad 2: /Stepper/pulY -> (no net)
- Q5 pad 2: /Stepper/dirY -> (no net)
- Q6 pad 2: /Stepper/enaY -> (no net)
- Q7 pad 2: /Stepper/pulZ -> (no net)
- Q8 pad 2: /Stepper/dirZ -> (no net)
- Q9 pad 2: /Stepper/enaZ -> (no net)
- XA1 pad D10: /Stepper/pulZ -> (no net)
- XA1 pad D12: /Stepper/pulY -> (no net)
- XA1 pad D24: /Stepper/dirY -> (no net)
- XA1 pad D25: /Stepper/enaY -> (no net)
- XA1 pad D26: /Stepper/dirZ -> (no net)
- XA1 pad D27: /Stepper/enaZ -> (no net)

Commit message: Add files via upload
Parts:
- removed j24: zMin, Connectors_Terminal_Blocks:TerminalBlock_Altech_AK300-2_P5.00mm
- added J24: gnd_+5v, Connectors_Terminal_Blocks:TerminalBlock_Altech_AK300-2_P5.00mm, F.Cu at (227.6, 24.4)
- added J28: +12v, Connectors_Terminal_Blocks:TerminalBlock_Altech_AK300-2_P5.00mm, F.Cu at (240.2, 24.3)
- added J29: LinActAnalog, Connectors_Terminal_Blocks:TerminalBlock_Altech_AK300-2_P5.00mm, F.Cu at (201.6, 24.3)
- added J30: LinActAnalog0, Connectors_Terminal_Blocks:TerminalBlock_Altech_AK300-2_P5.00mm, F.Cu at (214.5, 24.4)
- added J31: LinActDirection, Connectors_Terminal_Blocks:TerminalBlock_Altech_AK300-2_P5.00mm, F.Cu at (188.9, 24.1)
- added J32: zMin, Connectors_Terminal_Blocks:TerminalBlock_Altech_AK300-2_P5.00mm, F.Cu at (145.1, 24.5)
- added J33: +24V_source, Connectors_Terminal_Blocks:TerminalBlock_Altech_AK300-2_P5.00mm, F.Cu at (92.1, 76.1)
- added J34: +12V_source, Connectors_Terminal_Blocks:TerminalBlock_Altech_AK300-2_P5.00mm, F.Cu at (91.9, 101.8)
- J21: value +12V -> +5V_source
- XA1: moved to B.Cu
- moved J27 212.4 mm to (104.9, 24.3), turned to 0 degrees
- moved J9 201.3 mm to (117.8, 156.0), turned to 180 degrees
- moved R18 196.8 mm to (113.1, 146.4), turned to 90 degrees
- moved J26 191.1 mm to (118.4, 24.5), turned to 0 degrees
- moved J16 187.7 mm to (260.0, 156.1), turned to 180 degrees
- moved Q9 184.1 mm to (118.2, 142.5), turned to 0 degrees
- moved J8 182.9 mm to (130.5, 156.0), turned to 180 degrees
- moved R17 177.6 mm to (125.3, 146.6), turned to 90 degrees
- moved J25 172.1 mm to (131.7, 24.4), turned to 0 degrees
- moved J17 170.2 mm to (247.0, 156.1), turned to 180 degrees
- moved Q14 168.9 mm to (259.3, 142.8), turned to 0 degrees
- moved R7 167.2 mm to (255.1, 146.4), turned to 90 degrees
- moved J7 165.6 mm to (143.8, 156.0), turned to 180 degrees
- moved Q8 165.0 mm to (130.2, 142.5), turned to 0 degrees
- moved R16 157.3 mm to (139.2, 146.5), turned to 90 degrees
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Connections:
- J21 pad 1: Net-(J21-Pad1) -> +5V
- XA1 pad VIN: Net-(J21-Pad1) -> +12V
