File: ArduinoShield.sch (KiCad schematic (older format))
At the start: 1 part

Commit message: Add files via upload
Connections:
- net force/forceOut: now reaches XA1.A0
Changed lines of the file:
@@
 LIBS:contrib
 LIBS:valves
-LIBS:arduino
 LIBS:tennLogo
 LIBS:ArduinoShield-cache
@@
 	4800 5350 4950 5350
 $Comp
-L GND #PWR01
+L GND #PWR1
 U 1 1 5AC0DC4E
 P 4800 5450
-F 0 "#PWR01" H 4800 5200 50  0001 C CNN
+F 0 "#PWR1" H 4800 5200 50  0001 C CNN
 F 1 "GND" H 4800 5300 50  0000 C CNN
 F 2 "" H 4800 5450 50  0001 C CNN
@@
 NoConn ~ 4950 5850
 $Sheet
-S 1650 1000 1100 500
+S 800  3100 550  300
 U 5AC10749
 F0 "force" 60
 F1 "flexiForceSensor.sch" 60
+F2 "forceOut" I R 1350 3250 60
 $EndSheet
 $Sheet
-S 1800 2000 500  350
+S 800  2250 500  350
 U 5AC11210
 F0 "vfd" 60
 F1 "vfd.sch" 60
 $EndSheet
+Wire Wire Line
+	1350 3250 4950 3250
 $EndSCHEMATC

Commit message: Add files via upload
Connections:
- no-connect marks 8 -> 2
Changed lines of the file:
@@
 $Descr A4 11693 8268
 encoding utf-8
-Sheet 1 4
+Sheet 1 6
 Title ""
 Date ""
@@
 Comment4 ""
 $EndDescr
-$Comp
-L Arduino_Mega2560_Shield XA1
-U 1 1 5AC0677E
-P 6250 4100
-F 0 "XA1" V 6350 4100 60  0000 C CNN
-F 1 "Arduino_Mega2560_Shield" V 6150 4100 60  0000 C CNN
-F 2 "Arduino:Arduino_Mega2560_Shield" H 6950 6850 60  0001 C CNN
-F 3 "" H 6950 6850 60  0001 C CNN
-	1    6250 4100
-	1    0    0    -1
-$EndComp
 $Sheet
 S 10250 2900 550  1300
@@
 Wire Wire Line
 	7900 3650 7550 3650
-NoConn ~ 6000 1500
-NoConn ~ 6100 1500
-NoConn ~ 6200 1500
-NoConn ~ 6300 1500
-NoConn ~ 6400 1500
-NoConn ~ 6500 1500
 NoConn ~ 4950 5050
 Wire Wire Line
@@
 	4800 5350 4950 5350
 $Comp
-L GND #PWR1
+L GND #PWR01
 U 1 1 5AC0DC4E
 P 4800 5450
-F 0 "#PWR1" H 4800 5200 50  0001 C CNN
+F 0 "#PWR01" H 4800 5200 50  0001 C CNN
 F 1 "GND" H 4800 5300 50  0000 C CNN
 F 2 "" H 4800 5450 50  0001 C CNN
@@
 Wire Wire Line
 	1350 3250 4950 3250
+$Comp
+L Arduino_Mega2560_Shield XA1
+U 1 1 5AC0677E
+P 6250 4100
+F 0 "XA1" V 6350 4100 60  0000 C CNN
+F 1 "Arduino_Mega2560_Shield" V 6150 4100 60  0000 C CNN
+F 2 "Arduino:Arduino_Mega2560_Shield" H 6950 6850 60  0001 C CNN
+F 3 "" H 6950 6850 60  0001 C CNN
+	1    6250 4100
+	1    0    0    -1
+$EndComp
+$Sheet
+S 4050 600  550  600
+U 5ACC3536
+F0 "max6675" 60
+F1 "max6675.sch" 60
+$EndSheet
+$Sheet
+S 800  3650 600  400
+U 5ACC37CA
+F0 "ASC712" 60
+F1 "asc712.sch" 60
+$EndSheet
 $EndSCHEMATC

Commit message: Add files via upload
Parts:
- added J21: +12V, Connectors_Terminal_Blocks:TerminalBlock_Altech_AK300-2_P5.00mm, symbol Screw_Terminal_01x02
Connections:
- net GND: now also J21.2 (Pin_2)
- net +5V: now reaches XA1.5V1 (5V)
- net +5V: now also XA1.5V3 (5V), XA1.5V4 (5V)
- net at XA1.VIN: now also J21.1 (Pin_1)
Changed lines of the file:
@@
 F10 "enaZ" I L 10250 4050 60
+$EndSheet
+NoConn ~ 4950 5050
+$Comp
+L GND #PWR01
+U 1 1 5AC0DC4E
+P 4800 5450
+F 0 "#PWR01" H 4800 5200 50  0001 C CNN
+F 1 "GND" H 4800 5300 50  0000 C CNN
+F 2 "" H 4800 5450 50  0001 C CNN
+F 3 "" H 4800 5450 50  0001 C CNN
+	1    4800 5450
+	1    0    0    -1
+$EndComp
+NoConn ~ 4950 5850
+$Sheet
+S 800  3100 550  300
+U 5AC10749
+F0 "force" 60
+F1 "flexiForceSensor.sch" 60
+F2 "forceOut" I R 1350 3250 60
+$EndSheet
+$Sheet
+S 3200 5650 850  1050
+U 5AC11210
+F0 "vfd" 60
+F1 "vfd.sch" 60
+F2 "speedAnalogIn" I R 4050 5750 60
+F3 "Forward/Stop" I R 4050 5950 60
+F4 "Reverse/Stop" I R 4050 6150 60
+F5 "externalFault" I R 4050 6350 60
+F6 "jog" I R 4050 6500 60
+$EndSheet
+$Comp
+L Arduino_Mega2560_Shield XA1
+U 1 1 5AC0677E
+P 6250 4100
+F 0 "XA1" V 6350 4100 60  0000 C CNN
+F 1 "Arduino_Mega2560_Shield" V 6150 4100 60  0000 C CNN
+F 2 "Arduino:Arduino_Mega2560_Shield" H 6950 6850 60  0001 C CNN
+F 3 "" H 6950 6850 60  0001 C CNN
+	1    6250 4100
+	1    0    0    -1
+$EndComp
+$Sheet
+S 10300 5100 550  600
+U 5ACC3536
+F0 "max6675" 60
+F1 "max6675.sch" 60
+F2 "90" I L 10300 5550 60
+F3 "CS" I L 10300 5400 60
+F4 "SCK" I L 10300 5250 60
+$EndSheet
+$Sheet
+S 800  3600 600  400
+U 5ACC37CA
+F0 "ASC712" 60
+F1 "asc712.sch" 60
+F2 "currentSensor" I R 1400 3800 60
 $EndSheet
 Wire Wire Line
@@
 Wire Wire Line
 	7900 3650 7550 3650
-NoConn ~ 4950 5050
 Wire Wire Line
 	4950 5350 4950 5750
@@
 Wire Wire Line
 	4800 5350 4950 5350
+Wire Wire Line
+	4800 5450 4800 5350
+Connection ~ 4800 5350
+Wire Wire Line
+	1350 3250 4950 3250
 $Comp
-L GND #PWR01
-U 1 1 5AC0DC4E
-P 4800 5450
-F 0 "#PWR01" H 4800 5200 50  0001 C CNN
-F 1 "GND" H 4800 5300 50  0000 C CNN
-F 2 "" H 4800 5450 50  0001 C CNN
-F 3 "" H 4800 5450 50  0001 C CNN
-	1    4800 5450
+L Screw_Terminal_01x02 J21
+U 1 1 5ACF436B
+P 4800 6850
+F 0 "J21" H 4800 6950 50  0000 C CNN
+F 1 "+12V" H 4800 6650 50  0000 C CNN
+F 2 "Connectors_Terminal_Blocks:TerminalBlock_Altech_AK300-2_P5.00mm" H 4800 6850 50  0001 C CNN
+F 3 "" H 4800 6850 50  0001 C CNN
+	1    4800 6850
+	0    1    1    0
+$EndComp
+Wire Wire Line
+	4800 6650 4800 6250
+Wire Wire Line
+	4800 6250 4950 6250
+Wire Wire Line
+	4700 6650 4700 5750
+Wire Wire Line
+	4700 5750 4950 5750
+$Comp
+L +5V #PWR02
+U 1 1 5ACF49DF
+P 4800 5950
+F 0 "#PWR02" H 4800 5800 50  0001 C CNN
+F 1 "+5V" H 4800 6090 50  0000 C CNN
+F 2 "" H 4800 5950 50  0001 C CNN
+F 3 "" H 4800 5950 50  0001 C CNN
+	1    4800 5950
 	1    0    0    -1
 $EndComp
 Wire Wire Line
-	4800 5450 4800 5350
-Connection ~ 4800 5350
-NoConn ~ 4950 5850
-$Sheet
-S 800  3100 550  300
-U 5AC10749
-F0 "force" 60
-F1 "flexiForceSensor.sch" 60
-F2 "forceOut" I R 1350 3250 60
-$EndSheet
-$Sheet
-S 800  2250 500  350
-U 5AC11210
-F0 "vfd" 60
-F1 "vfd.sch" 60
-$EndSheet
+	4950 5950 4950 6150
+Connection ~ 4950 6050
 Wire Wire Line
-	1350 3250 4950 3250
-$Comp
-L Arduino_Mega2560_Shield XA1
-U 1 1 5AC0677E
-P 6250 4100
-F 0 "XA1" V 6350 4100 60  0000 C CNN
-F 1 "Arduino_Mega2560_Shield" V 6150 4100 60  0000 C CNN
-F 2 "Arduino:Arduino_Mega2560_Shield" H 6950 6850 60  0001 C CNN
-F 3 "" H 6950 6850 60  0001 C CNN
-	1    6250 4100
-	1    0    0    -1
-$EndComp
-$Sheet
-S 4050 600  550  600
-U 5ACC3536
-F0 "max6675" 60
-F1 "max6675.sch" 60
-$EndSheet
-$Sheet
-S 800  3650 600  400
-U 5ACC37CA
-F0 "ASC712" 60
-F1 "asc712.sch" 60
-$EndSheet
+	4950 5950 4800 5950
 $EndSCHEMATC

Commit message: Add files via upload
Connections:
- net Stepper/PulX: no longer XA1.D13
- net Stepper/dirX: no longer XA1.D22
- net Stepper/dirY: no longer XA1.D24
- net Stepper/dirZ: no longer XA1.D26
- net Stepper/enaX: no longer XA1.D23
- net Stepper/enaY: no longer XA1.D25
- net Stepper/enaZ: no longer XA1.D27
- net Stepper/pulY: no longer XA1.D12
- net Stepper/pulZ: no longer XA1.D10
Changed lines of the file:
@@
 $EndSheet
 $Sheet
-S 800  3600 600  400
+S 1400 5050 600  400
 U 5ACC37CA
 F0 "ASC712" 60
 F1 "asc712.sch" 60
-F2 "currentSensor" I R 1400 3800 60
+F2 "currentSensor" I R 2000 5250 60
 $EndSheet
 Wire Wire Line
-	7550 3050 10250 3050
-Wire Wire Line
-	10250 3450 8150 3450
-Wire Wire Line
-	8150 3450 8150 2950
-Wire Wire Line
-	8150 2950 7550 2950
-Wire Wire Line
-	10250 3850 8100 3850
-Wire Wire Line
-	8100 3850 8100 2750
-Wire Wire Line
-	8100 2750 7550 2750
-Wire Wire Line
-	10250 3150 7550 3150
-Wire Wire Line
-	10250 3250 7550 3250
-Wire Wire Line
-	10250 3550 10000 3550
-Wire Wire Line
-	10000 3550 10000 3350
-Wire Wire Line
-	10000 3350 7550 3350
-Wire Wire Line
-	10250 3650 8000 3650
-Wire Wire Line
-	8000 3650 8000 3450
-Wire Wire Line
-	8000 3450 7550 3450
-Wire Wire Line
-	10250 3950 9950 3950
-Wire Wire Line
-	9950 3950 9950 3550
-Wire Wire Line
-	9950 3550 7550 3550
-Wire Wire Line
-	10250 4050 7900 4050
-Wire Wire Line
-	7900 4050 7900 3650
-Wire Wire Line
-	7900 3650 7550 3650
-Wire Wire Line
 	4950 5350 4950 5750

Commit message: Add files via upload
Changed lines of the file:
@@
 $Descr A4 11693 8268
 encoding utf-8
-Sheet 1 6
+Sheet 1 7
 Title ""
 Date ""
@@
 $EndDescr
 $Sheet
-S 10250 2900 550  1300
+S 10300 1150 550  2400
 U 5AC0684B
 F0 "Stepper" 60
 F1 "stepperControl.sch" 60
-F2 "PulX" I L 10250 3050 60
-F3 "dirX" I L 10250 3150 60
-F4 "enaX" I L 10250 3250 60
-F5 "pulY" I L 10250 3450 60
-F6 "dirY" I L 10250 3550 60
-F7 "enaY" I L 10250 3650 60
-F8 "pulZ" I L 10250 3850 60
-F9 "dirZ" I L 10250 3950 60
-F10 "enaZ" I L 10250 4050 60
+F2 "pulY" I L 10300 2400 60
+F3 "dirY" I L 10300 2550 60
+F4 "enaY" I L 10300 2700 60
+F5 "pulZ" I L 10300 3050 60
+F6 "dirZ" I L 10300 3200 60
+F7 "enaZ" I L 10300 3350 60
+F8 "PulX1" I L 10300 1800 60
+F9 "dirX1" I L 10300 1950 60
+F10 "enaX1" I L 10300 2100 60
+F11 "PulX0" I L 10300 1300 60
+F12 "dirX0" I L 10300 1450 60
+F13 "enaX0" I L 10300 1600 60
 $EndSheet
 NoConn ~ 4950 5050
@@
 Wire Wire Line
 	4950 5950 4800 5950
+$Sheet
+S 9100 4650 500  1300
+U 5AD7D65A
+F0 "axis stops" 60
+F1 "file5AD7D659.sch" 60
+$EndSheet
 $EndSCHEMATC

Commit message: Add files via upload
Changed lines of the file:
@@
 $Descr A4 11693 8268
 encoding utf-8
-Sheet 1 7
+Sheet 1 8
 Title ""
 Date ""
@@
 NoConn ~ 4950 5050
 $Comp
-L GND #PWR01
+L GND #PWR1
 U 1 1 5AC0DC4E
 P 4800 5450
-F 0 "#PWR01" H 4800 5200 50  0001 C CNN
+F 0 "#PWR1" H 4800 5200 50  0001 C CNN
 F 1 "GND" H 4800 5300 50  0000 C CNN
 F 2 "" H 4800 5450 50  0001 C CNN
@@
 $EndSheet
 $Sheet
-S 3200 5650 850  1050
+S 5650 6850 1050 850
 U 5AC11210
 F0 "vfd" 60
 F1 "vfd.sch" 60
-F2 "speedAnalogIn" I R 4050 5750 60
-F3 "Forward/Stop" I R 4050 5950 60
-F4 "Reverse/Stop" I R 4050 6150 60
-F5 "externalFault" I R 4050 6350 60
-F6 "jog" I R 4050 6500 60
+F2 "speedAnalogIn" I T 5750 6850 60
+F3 "Forward/Stop" I T 5950 6850 60
+F4 "Reverse/Stop" I T 6150 6850 60
+F5 "externalFault" I T 6350 6850 60
+F6 "jog" I T 6500 6850 60
 $EndSheet
 $Comp
@@
 $EndSheet
 $Sheet
-S 1400 5050 600  400
+S 850  3550 600  400
 U 5ACC37CA
 F0 "ASC712" 60
 F1 "asc712.sch" 60
-F2 "currentSensor" I R 2000 5250 60
+F2 "currentSensor" I R 1450 3750 60
 $EndSheet
 Wire Wire Line
@@
 	4700 5750 4950 5750
 $Comp
-L +5V #PWR02
+L +5V #PWR2
 U 1 1 5ACF49DF
 P 4800 5950
-F 0 "#PWR02" H 4800 5800 50  0001 C CNN
+F 0 "#PWR2" H 4800 5800 50  0001 C CNN
 F 1 "+5V" H 4800 6090 50  0000 C CNN
 F 2 "" H 4800 5950 50  0001 C CNN
@@
 	4950 5950 4800 5950
 $Sheet
-S 9100 4650 500  1300
+S 9100 4650 550  1100
 U 5AD7D65A
 F0 "axis stops" 60
 F1 "file5AD7D659.sch" 60
+F2 "xMin" I L 9100 4800 60
+F3 "xMax" I L 9100 4900 60
+F4 "zMin" I L 9100 5100 60
+F5 "zMax" I L 9100 5200 60
+F6 "yMin" I L 9100 5450 60
+F7 "yMax" I L 9100 5600 60
+$EndSheet
+$Sheet
+S 1350 5700 500  1000
+U 5AD82948
+F0 "linearAct" 60
+F1 "file5AD82947.sch" 60
 $EndSheet
 $EndSCHEMATC

Commit message: Add files via upload
Parts:
- removed J21: +12V, Connectors_Terminal_Blocks:TerminalBlock_Altech_AK300-2_P5.00mm, symbol Screw_Terminal_01x02
Connections:
- net +12V: now reaches XA1.VIN
Changed lines of the file:
@@
 $EndDescr
 $Sheet
-S 10300 1150 550  2400
+S 9150 950  550  2400
 U 5AC0684B
 F0 "Stepper" 60
 F1 "stepperControl.sch" 60
-F2 "pulY" I L 10300 2400 60
-F3 "dirY" I L 10300 2550 60
-F4 "enaY" I L 10300 2700 60
-F5 "pulZ" I L 10300 3050 60
-F6 "dirZ" I L 10300 3200 60
-F7 "enaZ" I L 10300 3350 60
-F8 "PulX1" I L 10300 1800 60
-F9 "dirX1" I L 10300 1950 60
-F10 "enaX1" I L 10300 2100 60
-F11 "PulX0" I L 10300 1300 60
-F12 "dirX0" I L 10300 1450 60
-F13 "enaX0" I L 10300 1600 60
+F2 "pulY" I L 9150 2200 60
+F3 "dirY" I L 9150 2350 60
+F4 "enaY" I L 9150 2500 60
+F5 "pulZ" I L 9150 2850 60
+F6 "dirZ" I L 9150 3000 60
+F7 "enaZ" I L 9150 3150 60
+F8 "PulX1" I L 9150 1600 60
+F9 "dirX1" I L 9150 1750 60
+F10 "enaX1" I L 9150 1900 60
+F11 "PulX0" I L 9150 1100 60
+F12 "dirX0" I L 9150 1250 60
+F13 "enaX0" I L 9150 1400 60
 $EndSheet
 NoConn ~ 4950 5050
 $Comp
-L GND #PWR1
+L GND #PWR2
 U 1 1 5AC0DC4E
 P 4800 5450
-F 0 "#PWR1" H 4800 5200 50  0001 C CNN
+F 0 "#PWR2" H 4800 5200 50  0001 C CNN
 F 1 "GND" H 4800 5300 50  0000 C CNN
 F 2 "" H 4800 5450 50  0001 C CNN
@@
 	1350 3250 4950 3250
 $Comp
-L Screw_Terminal_01x02 J21
-U 1 1 5ACF436B
-P 4800 6850
-F 0 "J21" H 4800 6950 50  0000 C CNN
-F 1 "+12V" H 4800 6650 50  0000 C CNN
-F 2 "Connectors_Terminal_Blocks:TerminalBlock_Altech_AK300-2_P5.00mm" H 4800 6850 50  0001 C CNN
-F 3 "" H 4800 6850 50  0001 C CNN
-	1    4800 6850
-	0    1    1    0
-$EndComp
-Wire Wire Line
-	4800 6650 4800 6250
-Wire Wire Line
-	4800 6250 4950 6250
-Wire Wire Line
-	4700 6650 4700 5750
-Wire Wire Line
-	4700 5750 4950 5750
-$Comp
-L +5V #PWR2
+L +5V #PWR3
 U 1 1 5ACF49DF
 P 4800 5950
-F 0 "#PWR2" H 4800 5800 50  0001 C CNN
+F 0 "#PWR3" H 4800 5800 50  0001 C CNN
 F 1 "+5V" H 4800 6090 50  0000 C CNN
 F 2 "" H 4800 5950 50  0001 C CNN
@@
 	4950 5950 4800 5950
 $Sheet
-S 9100 4650 550  1100
-U 5AD7D65A
-F0 "axis stops" 60
-F1 "file5AD7D659.sch" 60
-F2 "xMin" I L 9100 4800 60
-F3 "xMax" I L 9100 4900 60
-F4 "zMin" I L 9100 5100 60
-F5 "zMax" I L 9100 5200 60
-F6 "yMin" I L 9100 5450 60
-F7 "yMax" I L 9100 5600 60
-$EndSheet
-$Sheet
 S 1350 5700 500  1000
 U 5AD82948
@@
 F1 "file5AD82947.sch" 60
 $EndSheet
+$Comp
+L +12V #PWR1
+U 1 1 5AD8E9B3
+P 4700 6250
+F 0 "#PWR1" H 4700 6100 50  0001 C CNN
+F 1 "+12V" H 4700 6390 50  0000 C CNN
+F 2 "" H 4700 6250 50  0001 C CNN
+F 3 "" H 4700 6250 50  0001 C CNN
+	1    4700 6250
+	1    0    0    -1
+$EndComp
+Wire Wire Line
+	4950 6250 4700 6250
+$Sheet
+S 3550 6700 650  800
+U 5AD8F2C1
+F0 "power" 60
+F1 "power.sch" 60
+$EndSheet
 $EndSCHEMATC
