File: asc712.sch (KiCad schematic (older format))
At the start: 0 parts

Commit message: Add files via upload
Parts:
- added J20: ASC712, Socket_Strips:Socket_Strip_Straight_1x03_Pitch2.54mm, symbol Conn_01x03_Female
Connections:
- new net +5V: J20.3 (Pin_3)
- new net GND: J20.1 (Pin_1)
- new net currentSensor: J20.2 (Pin_2)
Changed lines of the file:
@@
 Comment4 ""
 $EndDescr
+$Comp
+L Conn_01x03_Female J20
+U 1 1 5ACF2120
+P 5200 4200
+F 0 "J20" H 5200 4400 50  0000 C CNN
+F 1 "ASC712" H 5200 4000 50  0000 C CNN
+F 2 "Socket_Strips:Socket_Strip_Straight_1x03_Pitch2.54mm" H 5200 4200 50  0001 C CNN
+F 3 "" H 5200 4200 50  0001 C CNN
+	1    5200 4200
+	1    0    0    -1
+$EndComp
+$Comp
+L GND #PWR013
+U 1 1 5ACF2153
+P 4950 4100
+F 0 "#PWR013" H 4950 3850 50  0001 C CNN
+F 1 "GND" H 4950 3950 50  0000 C CNN
+F 2 "" H 4950 4100 50  0001 C CNN
+F 3 "" H 4950 4100 50  0001 C CNN
+	1    4950 4100
+	0    1    1    0
+$EndComp
+$Comp
+L +5V #PWR014
+U 1 1 5ACF217A
+P 4900 4300
+F 0 "#PWR014" H 4900 4150 50  0001 C CNN
+F 1 "+5V" H 4900 4440 50  0000 C CNN
+F 2 "" H 4900 4300 50  0001 C CNN
+F 3 "" H 4900 4300 50  0001 C CNN
+	1    4900 4300
+	-1   0    0    1
+$EndComp
+Text HLabel 4550 4200 0    60   Input ~ 0
+currentSensor
+Wire Wire Line
+	5000 4100 4950 4100
+Wire Wire Line
+	5000 4300 4900 4300
+Wire Wire Line
+	5000 4200 4550 4200
 $EndSCHEMATC
