File: file5AD7D659.sch (KiCad schematic (older format))
At the start: 6 parts

Commit message: Add files via upload
Parts:
- J22: renamed from J?; value Screw_Terminal_01x02 -> xMin; footprint (none) -> Connectors_Terminal_Blocks:TerminalBlock_Altech_AK300-2_P5.00mm
- J23: renamed from J?; value Screw_Terminal_01x02 -> xMax; footprint (none) -> Connectors_Terminal_Blocks:TerminalBlock_Altech_AK300-2_P5.00mm
- J25: renamed from J?; value Screw_Terminal_01x02 -> zMax; footprint (none) -> Connectors_Terminal_Blocks:TerminalBlock_Altech_AK300-2_P5.00mm
- J26: renamed from J?; value Screw_Terminal_01x02 -> yMin; footprint (none) -> Connectors_Terminal_Blocks:TerminalBlock_Altech_AK300-2_P5.00mm
- J27: renamed from J?; value Screw_Terminal_01x02 -> yMax; footprint (none) -> Connectors_Terminal_Blocks:TerminalBlock_Altech_AK300-2_P5.00mm
- j24: renamed from J?; value Screw_Terminal_01x02 -> zMin; footprint (none) -> Connectors_Terminal_Blocks:TerminalBlock_Altech_AK300-2_P5.00mm
Changed lines of the file:
@@
 $Descr A4 11693 8268
 encoding utf-8
-Sheet 7 7
+Sheet 7 8
 Title ""
 Date ""
@@
 $EndDescr
 $Comp
-L Screw_Terminal_01x02 J?
+L Screw_Terminal_01x02 J22
 U 1 1 5AD7D6AD
 P 3100 2100
-F 0 "J?" H 3100 2200 50  0000 C CNN
-F 1 "Screw_Terminal_01x02" H 3100 1900 50  0000 C CNN
-F 2 "" H 3100 2100 50  0001 C CNN
+F 0 "J22" H 3100 2200 50  0000 C CNN
+F 1 "xMin" H 3100 1900 50  0000 C CNN
+F 2 "Connectors_Terminal_Blocks:TerminalBlock_Altech_AK300-2_P5.00mm" H 3100 2100 50  0001 C CNN
 F 3 "" H 3100 2100 50  0001 C CNN
 	1    3100 2100
@@
 $EndComp
 $Comp
-L Screw_Terminal_01x02 J?
+L Screw_Terminal_01x02 J23
 U 1 1 5AD7D8CF
 P 3850 2100
-F 0 "J?" H 3850 2200 50  0000 C CNN
-F 1 "Screw_Terminal_01x02" H 3850 1900 50  0000 C CNN
-F 2 "" H 3850 2100 50  0001 C CNN
+F 0 "J23" H 3850 2200 50  0000 C CNN
+F 1 "xMax" H 3850 1900 50  0000 C CNN
+F 2 "Connectors_Terminal_Blocks:TerminalBlock_Altech_AK300-2_P5.00mm" H 3850 2100 50  0001 C CNN
 F 3 "" H 3850 2100 50  0001 C CNN
 	1    3850 2100
@@
 $EndComp
 $Comp
-L Screw_Terminal_01x02 J?
+L Screw_Terminal_01x02 j24
 U 1 1 5AD7DA82
 P 4650 2050
-F 0 "J?" H 4650 2150 50  0000 C CNN
-F 1 "Screw_Terminal_01x02" H 4650 1850 50  0000 C CNN
-F 2 "" H 4650 2050 50  0001 C CNN
+F 0 "j24" H 4650 2150 50  0000 C CNN
+F 1 "zMin" H 4650 1850 50  0000 C CNN
+F 2 "Connectors_Terminal_Blocks:TerminalBlock_Altech_AK300-2_P5.00mm" H 4650 2050 50  0001 C CNN
 F 3 "" H 4650 2050 50  0001 C CNN
 	1    4650 2050
@@
 $EndComp
 $Comp
-L Screw_Terminal_01x02 J?
+L Screw_Terminal_01x02 J25
 U 1 1 5AD7DA88
 P 5400 2050
-F 0 "J?" H 5400 2150 50  0000 C CNN
-F 1 "Screw_Terminal_01x02" H 5400 1850 50  0000 C CNN
-F 2 "" H 5400 2050 50  0001 C CNN
+F 0 "J25" H 5400 2150 50  0000 C CNN
+F 1 "zMax" H 5400 1850 50  0000 C CNN
+F 2 "Connectors_Terminal_Blocks:TerminalBlock_Altech_AK300-2_P5.00mm" H 5400 2050 50  0001 C CNN
 F 3 "" H 5400 2050 50  0001 C CNN
 	1    5400 2050
@@
 $EndComp
 $Comp
-L Screw_Terminal_01x02 J?
+L Screw_Terminal_01x02 J26
 U 1 1 5AD7DABC
 P 6200 2100
-F 0 "J?" H 6200 2200 50  0000 C CNN
-F 1 "Screw_Terminal_01x02" H 6200 1900 50  0000 C CNN
-F 2 "" H 6200 2100 50  0001 C CNN
+F 0 "J26" H 6200 2200 50  0000 C CNN
+F 1 "yMin" H 6200 1900 50  0000 C CNN
+F 2 "Connectors_Terminal_Blocks:TerminalBlock_Altech_AK300-2_P5.00mm" H 6200 2100 50  0001 C CNN
 F 3 "" H 6200 2100 50  0001 C CNN
 	1    6200 2100
@@
 $EndComp
 $Comp
-L Screw_Terminal_01x02 J?
+L Screw_Terminal_01x02 J27
 U 1 1 5AD7DAC2
 P 6950 2100
-F 0 "J?" H 6950 2200 50  0000 C CNN
-F 1 "Screw_Terminal_01x02" H 6950 1900 50  0000 C CNN
-F 2 "" H 6950 2100 50  0001 C CNN
+F 0 "J27" H 6950 2200 50  0000 C CNN
+F 1 "yMax" H 6950 1900 50  0000 C CNN
+F 2 "Connectors_Terminal_Blocks:TerminalBlock_Altech_AK300-2_P5.00mm" H 6950 2100 50  0001 C CNN
 F 3 "" H 6950 2100 50  0001 C CNN
 	1    6950 2100
@@
 Connection ~ 6200 2600
 $Comp
-L +5V #PWR?
+L +5V #PWR15
 U 1 1 5AD7DF62
 P 2600 2500
-F 0 "#PWR?" H 2600 2350 50  0001 C CNN
+F 0 "#PWR15" H 2600 2350 50  0001 C CNN
 F 1 "+5V" H 2600 2640 50  0000 C CNN
 F 2 "" H 2600 2500 50  0001 C CNN

Commit message: Add files via upload
Parts:
- renumbered j24 to J32
Changed lines of the file:
@@
 $Descr A4 11693 8268
 encoding utf-8
-Sheet 7 8
+Sheet 7 9
 Title ""
 Date ""
@@
 $EndComp
 $Comp
-L Screw_Terminal_01x02 j24
+L Screw_Terminal_01x02 J32
 U 1 1 5AD7DA82
 P 4650 2050
-F 0 "j24" H 4650 2150 50  0000 C CNN
+F 0 "J32" H 4650 2200 50  0000 C CNN
 F 1 "zMin" H 4650 1850 50  0000 C CNN
 F 2 "Connectors_Terminal_Blocks:TerminalBlock_Altech_AK300-2_P5.00mm" H 4650 2050 50  0001 C CNN
@@
 Connection ~ 6200 2600
 $Comp
-L +5V #PWR15
+L +5V #PWR016
 U 1 1 5AD7DF62
 P 2600 2500
-F 0 "#PWR15" H 2600 2350 50  0001 C CNN
+F 0 "#PWR016" H 2600 2350 50  0001 C CNN
 F 1 "+5V" H 2600 2640 50  0000 C CNN
 F 2 "" H 2600 2500 50  0001 C CNN
