File: file5AD82947.sch (KiCad schematic (older format))
At the start: 5 parts, among them J24 gnd +5v, J28 +12v, J29 Screw_Terminal_01x02, J30 Screw_Terminal_01x02, J31 Screw_Terminal_01x02

Commit message: Add files via upload
Parts:
- J24: value gnd +5v -> gnd_+5v; footprint (none) -> Connectors_Terminal_Blocks:TerminalBlock_Altech_AK300-2_P5.00mm
- J28: footprint (none) -> Connectors_Terminal_Blocks:TerminalBlock_Altech_AK300-2_P5.00mm
- J29: value Screw_Terminal_01x02 -> LinActAnalog; footprint (none) -> Connectors_Terminal_Blocks:TerminalBlock_Altech_AK300-2_P5.00mm
- J30: value Screw_Terminal_01x02 -> LinActAnalog0; footprint (none) -> Connectors_Terminal_Blocks:TerminalBlock_Altech_AK300-2_P5.00mm
- J31: value Screw_Terminal_01x02 -> LinActDirection; footprint (none) -> Connectors_Terminal_Blocks:TerminalBlock_Altech_AK300-2_P5.00mm
Changed lines of the file:
@@
 P 3550 2250
 F 0 "J24" H 3550 2350 50  0000 C CNN
-F 1 "gnd +5v" V 3750 2150 50  0000 C CNN
-F 2 "" H 3550 2250 50  0001 C CNN
+F 1 "gnd_+5v" V 3750 2150 50  0000 C CNN
+F 2 "Connectors_Terminal_Blocks:TerminalBlock_Altech_AK300-2_P5.00mm" H 3550 2250 50  0001 C CNN
 F 3 "" H 3550 2250 50  0001 C CNN
 	1    3550 2250
@@
 $EndComp
 $Comp
-L GND #PWR16
+L GND #PWR28
 U 1 1 5AD829D6
 P 3550 2650
-F 0 "#PWR16" H 3550 2400 50  0001 C CNN
+F 0 "#PWR28" H 3550 2400 50  0001 C CNN
 F 1 "GND" H 3550 2500 50  0000 C CNN
 F 2 "" H 3550 2650 50  0001 C CNN
@@
 $EndComp
 $Comp
-L +5V #PWR17
+L +5V #PWR29
 U 1 1 5AD829EF
 P 3750 2600
-F 0 "#PWR17" H 3750 2450 50  0001 C CNN
+F 0 "#PWR29" H 3750 2450 50  0001 C CNN
 F 1 "+5V" H 3750 2740 50  0000 C CNN
 F 2 "" H 3750 2600 50  0001 C CNN
@@
 P 4200 2250
 F 0 "J28" H 4200 2350 50  0000 C CNN
-F 1 "+12v" V 4350 1850 50  0000 C CNN
-F 2 "" H 4200 2250 50  0001 C CNN
+F 1 "+12v" V 4350 2200 50  0000 C CNN
+F 2 "Connectors_Terminal_Blocks:TerminalBlock_Altech_AK300-2_P5.00mm" H 4200 2250 50  0001 C CNN
 F 3 "" H 4200 2250 50  0001 C CNN
 	1    4200 2250
@@
 $EndComp
 $Comp
-L +12V #PWR19
+L +12V #PWR31
 U 1 1 5AD82A48
 P 4300 2550
-F 0 "#PWR19" H 4300 2400 50  0001 C CNN
+F 0 "#PWR31" H 4300 2400 50  0001 C CNN
 F 1 "+12V" H 4300 2690 50  0000 C CNN
 F 2 "" H 4300 2550 50  0001 C CNN
@@
 P 5250 2350
 F 0 "J29" H 5250 2450 50  0000 C CNN
-F 1 "Screw_Terminal_01x02" H 5250 2150 50  0000 C CNN
-F 2 "" H 5250 2350 50  0001 C CNN
+F 1 "LinActAnalog" H 5250 2150 50  0000 C CNN
+F 2 "Connectors_Terminal_Blocks:TerminalBlock_Altech_AK300-2_P5.00mm" H 5250 2350 50  0001 C CNN
 F 3 "" H 5250 2350 50  0001 C CNN
 	1    5250 2350
@@
 P 5700 2350
 F 0 "J30" H 5700 2450 50  0000 C CNN
-F 1 "Screw_Terminal_01x02" H 5700 2150 50  0000 C CNN
-F 2 "" H 5700 2350 50  0001 C CNN
+F 1 "LinActAnalog0" H 5700 2150 50  0000 C CNN
+F 2 "Connectors_Terminal_Blocks:TerminalBlock_Altech_AK300-2_P5.00mm" H 5700 2350 50  0001 C CNN
 F 3 "" H 5700 2350 50  0001 C CNN
 	1    5700 2350
@@
 $EndComp
 $Comp
-L +5V #PWR20
+L +5V #PWR32
 U 1 1 5AD82B1D
 P 5250 2800
-F 0 "#PWR20" H 5250 2650 50  0001 C CNN
+F 0 "#PWR32" H 5250 2650 50  0001 C CNN
 F 1 "+5V" H 5250 2940 50  0000 C CNN
 F 2 "" H 5250 2800 50  0001 C CNN
@@
 $EndComp
 $Comp
-L GND #PWR21
+L GND #PWR33
 U 1 1 5AD82B39
 P 5800 2850
-F 0 "#PWR21" H 5800 2600 50  0001 C CNN
+F 0 "#PWR33" H 5800 2600 50  0001 C CNN
 F 1 "GND" H 5800 2700 50  0000 C CNN
 F 2 "" H 5800 2850 50  0001 C CNN
@@
 	5500 3150 5300 3150
 $Comp
-L GND #PWR18
+L GND #PWR30
 U 1 1 5AD82C9B
 P 4100 2600
-F 0 "#PWR18" H 4100 2350 50  0001 C CNN
+F 0 "#PWR30" H 4100 2350 50  0001 C CNN
 F 1 "GND" H 4100 2450 50  0000 C CNN
 F 2 "" H 4100 2600 50  0001 C CNN
@@
 P 6750 2400
 F 0 "J31" H 6750 2500 50  0000 C CNN
-F 1 "Screw_Terminal_01x02" H 6750 2200 50  0000 C CNN
-F 2 "" H 6750 2400 50  0001 C CNN
+F 1 "LinActDirection" H 6750 2200 50  0000 C CNN
+F 2 "Connectors_Terminal_Blocks:TerminalBlock_Altech_AK300-2_P5.00mm" H 6750 2400 50  0001 C CNN
 F 3 "" H 6750 2400 50  0001 C CNN
 	1    6750 2400
