File: flexiForceSensor.sch (KiCad schematic (older format))
At the start: 0 parts

Commit message: Add files via upload
Parts:
- added C1, C5: C, symbol C
- added C2, C3, C4, C6, C7: CP, symbol CP
- added D1, D2: D, symbol D
- added J10: Flex_Sensor, symbol Screw_Terminal_01x02
- added R1, R2, R3, R4: R, symbol R
- added RV1, RV2: POT, symbol POT
- added U1: NE555, Housings_DIP:DIP-8_W7.62mm_Socket_LongPads, symbol NE555
- added U2: LM337_TO220, TO_SOT_Packages_THT:TO-220_Vertical, symbol LM337_TO220
- added U3: MCP6004, symbol MCP6004
Connections:
- new net: C2.1, R2.2, U1.2 (TR), U1.6 (THR)
- new net: C3.2, U1.3 (Q)
- new net: C1.1, U1.5 (CV)
- new net: R1.2, R2.1, U1.7 (DIS)
- new net: R3.1, RV1.1, U2.1 (ADJ)
- new net: C4.2, D2.2 (A), U2.2 (VI)
- new net: C7.2, R3.2, R4.1, U2.3 (VO)
- new net: C4.1, C7.1, RV1.2, RV1.3
- new net: D1.2 (A), D2.1 (K)
- new net: C5.2, C6.2, J10.2 (Pin_2), R4.2
- new net: C5.1, J10.1 (Pin_1), RV2.3, U3.2 (-)
- new net +12V: R1.1, U1.4 (R), U1.8 (VCC)
- new net +5V: U3.11 (V-)
- new net GND: C1.2, C2.2, C6.1, D1.1 (K), U1.1 (GND), U3.3 (+), U3.4 (V+)
- new net forceOut: RV2.1, RV2.2, U3.1

Commit message: Add files via upload
Parts:
- C1: footprint (none) -> Capacitors_THT:C_Disc_D6.0mm_W2.5mm_P5.00mm
- C2: footprint (none) -> Capacitors_THT:CP_Radial_D4.0mm_P1.50mm
- C3: footprint (none) -> Capacitors_THT:CP_Radial_D5.0mm_P2.00mm
- D1, D2: footprint (none) -> Diodes_THT:D_DO-35_SOD27_P7.62mm_Horizontal
- J10: footprint (none) -> Connectors_Terminal_Blocks:TerminalBlock_Altech_AK300-2_P5.00mm
- R1, R2, R3, R4: footprint (none) -> Resistors_THT:R_Axial_DIN0207_L6.3mm_D2.5mm_P10.16mm_Horizontal
- RV1, RV2: footprint (none) -> Potentiometers:Potentiometer_WirePads_largePads
- U2: footprint TO_SOT_Packages_THT:TO-220_Vertical -> TO_SOT_Packages_THT:TO-220-3_Vertical
- U3: footprint (none) -> Housings_DIP:DIP-8_W10.16mm_LongPads
Connections:
- net at C3.1: now also D1.2 (A), D2.1 (K)
Changed lines of the file:
@@
 F 0 "C1" H 11225 11950 50  0000 L CNN
 F 1 "C" H 11225 11750 50  0000 L CNN
-F 2 "" H 11238 11700 50  0001 C CNN
+F 2 "Capacitors_THT:C_Disc_D6.0mm_W2.5mm_P5.00mm" H 11238 11700 50  0001 C CNN
 F 3 "" H 11200 11850 50  0001 C CNN
 	1    11200 11850
@@
 $EndComp
 $Comp
-L +12V #PWR04
+L +12V #PWR05
 U 1 1 5AC3C707
 P 12500 10550
-F 0 "#PWR04" H 12500 10400 50  0001 C CNN
+F 0 "#PWR05" H 12500 10400 50  0001 C CNN
 F 1 "+12V" H 12500 10690 50  0000 C CNN
 F 2 "" H 12500 10550 50  0001 C CNN
@@
 F 0 "C3" H 14825 11050 50  0000 L CNN
 F 1 "CP" H 14825 10850 50  0000 L CNN
-F 2 "" H 14838 10800 50  0001 C CNN
+F 2 "Capacitors_THT:CP_Radial_D5.0mm_P2.00mm" H 14838 10800 50  0001 C CNN
 F 3 "" H 14800 10950 50  0001 C CNN
 	1    14800 10950
@@
 F 0 "C2" H 13875 12250 50  0000 L CNN
 F 1 "CP" H 13875 12050 50  0000 L CNN
-F 2 "" H 13888 12000 50  0001 C CNN
+F 2 "Capacitors_THT:CP_Radial_D4.0mm_P1.50mm" H 13888 12000 50  0001 C CNN
 F 3 "" H 13850 12150 50  0001 C CNN
 	1    13850 12150
@@
 F 0 "R1" V 13930 11350 50  0000 C CNN
 F 1 "R" V 13850 11350 50  0000 C CNN
-F 2 "" V 13780 11350 50  0001 C CNN
+F 2 "Resistors_THT:R_Axial_DIN0207_L6.3mm_D2.5mm_P10.16mm_Horizontal" V 13780 11350 50  0001 C CNN
 F 3 "" H 13850 11350 50  0001 C CNN
 	1    13850 11350
@@
 F 0 "R2" V 13930 11750 50  0000 C CNN
 F 1 "R" V 13850 11750 50  0000 C CNN
-F 2 "" V 13780 11750 50  0001 C CNN
+F 2 "Resistors_THT:R_Axial_DIN0207_L6.3mm_D2.5mm_P10.16mm_Horizontal" V 13780 11750 50  0001 C CNN
 F 3 "" H 13850 11750 50  0001 C CNN
 	1    13850 11750
@@
 F 0 "U2" H 17300 10825 50  0000 C CNN
 F 1 "LM337_TO220" H 17450 10825 50  0000 L CNN
-F 2 "TO_SOT_Packages_THT:TO-220_Vertical" H 17450 10750 50  0001 C CIN
+F 2 "TO_SOT_Packages_THT:TO-220-3_Vertical" H 17450 10750 50  0001 C CIN
 F 3 "" H 17450 10950 50  0001 C CNN
 	1    17450 10950
@@
 F 0 "D2" H 16250 11050 50  0000 C CNN
 F 1 "D" H 16250 10850 50  0000 C CNN
-F 2 "" H 16250 10950 50  0001 C CNN
+F 2 "Diodes_THT:D_DO-35_SOD27_P7.62mm_Horizontal" H 16250 10950 50  0001 C CNN
 F 3 "" H 16250 10950 50  0001 C CNN
 	1    16250 10950
@@
 F 0 "D1" H 15500 11750 50  0000 C CNN
 F 1 "D" H 15500 11550 50  0000 C CNN
-F 2 "" H 15500 11650 50  0001 C CNN
+F 2 "Diodes_THT:D_DO-35_SOD27_P7.62mm_Horizontal" H 15500 11650 50  0001 C CNN
 F 3 "" H 15500 11650 50  0001 C CNN
 	1    15500 11650
@@
 F 0 "RV1" V 18025 10250 50  0000 C CNN
 F 1 "POT" V 18100 10250 50  0000 C CNN
-F 2 "" H 18200 10250 50  0001 C CNN
+F 2 "Potentiometers:Potentiometer_WirePads_largePads" H 18200 10250 50  0001 C CNN
 F 3 "" H 18200 10250 50  0001 C CNN
 	1    18200 10250
@@
 F 0 "R3" V 18280 10750 50  0000 C CNN
 F 1 "R" V 18200 10750 50  0000 C CNN
-F 2 "" V 18130 10750 50  0001 C CNN
+F 2 "Resistors_THT:R_Axial_DIN0207_L6.3mm_D2.5mm_P10.16mm_Horizontal" V 18130 10750 50  0001 C CNN
 F 3 "" H 18200 10750 50  0001 C CNN
 	1    18200 10750
@@
 $EndComp
 $Comp
-L GND #PWR05
+L GND #PWR06
 U 1 1 5AC407D3
 P 12450 12500
-F 0 "#PWR05" H 12450 12250 50  0001 C CNN
+F 0 "#PWR06" H 12450 12250 50  0001 C CNN
 F 1 "GND" H 12450 12350 50  0000 C CNN
 F 2 "" H 12450 12500 50  0001 C CNN
@@
 F 0 "R4" V 18630 11550 50  0000 C CNN
 F 1 "R" V 18550 11550 50  0000 C CNN
-F 2 "" V 18480 11550 50  0001 C CNN
+F 2 "Resistors_THT:R_Axial_DIN0207_L6.3mm_D2.5mm_P10.16mm_Horizontal" V 18480 11550 50  0001 C CNN
 F 3 "" H 18550 11550 50  0001 C CNN
 	1    18550 11550
@@
 	13850 12400 13850 12300
 Wire Wire Line
-	15000 10950 16100 10950
+	14950 10950 16100 10950
 Wire Wire Line
 	15500 10950 15500 11500
@@
 F 0 "U3" H 19250 14300 50  0000 L CNN
 F 1 "MCP6004" H 19250 13900 50  0000 L CNN
-F 2 "" H 19200 14200 50  0001 C CNN
+F 2 "Housings_DIP:DIP-8_W10.16mm_LongPads" H 19200 14200 50  0001 C CNN
 F 3 "" H 19300 14300 50  0001 C CNN
 	1    19250 14100
@@
 F 0 "J10" H 17800 14950 50  0000 C CNN
 F 1 "Flex_Sensor" H 17800 14650 50  0000 C CNN
-F 2 "" H 17800 14850 50  0001 C CNN
+F 2 "Connectors_Terminal_Blocks:TerminalBlock_Altech_AK300-2_P5.00mm" H 17800 14850 50  0001 C CNN
 F 3 "" H 17800 14850 50  0001 C CNN
 	1    17800 14850
@@
 	19150 13150 19700 13150
 $Comp
-L +5V #PWR06
+L +5V #PWR07
 U 1 1 5AC47E2C
 P 19500 14850
-F 0 "#PWR06" H 19500 14700 50  0001 C CNN
+F 0 "#PWR07" H 19500 14700 50  0001 C CNN
 F 1 "+5V" H 19500 14990 50  0000 C CNN
 F 2 "" H 19500 14850 50  0001 C CNN
@@
 $EndComp
 $Comp
-L GND #PWR07
+L GND #PWR08
 U 1 1 5AC47EC1
 P 19700 13250
-F 0 "#PWR07" H 19700 13000 50  0001 C CNN
+F 0 "#PWR08" H 19700 13000 50  0001 C CNN
 F 1 "GND" H 19700 13100 50  0000 C CNN
 F 2 "" H 19700 13250 50  0001 C CNN
@@
 F 0 "RV2" V 19025 15450 50  0000 C CNN
 F 1 "POT" V 19100 15450 50  0000 C CNN
-F 2 "" H 19200 15450 50  0001 C CNN
+F 2 "Potentiometers:Potentiometer_WirePads_largePads" H 19200 15450 50  0001 C CNN
 F 3 "" H 19200 15450 50  0001 C CNN
 	1    19200 15450
