File: max6675.sch (KiCad schematic (older format))
At the start: 0 parts

Commit message: Add files via upload
Parts:
- added J19: MAX6675, Socket_Strips:Socket_Strip_Straight_1x05_Pitch2.54mm, symbol Conn_01x05_Female
Connections:
- new net +5V: J19.2 (Pin_2)
- new net 90: J19.3 (Pin_3)
- new net CS: J19.4 (Pin_4)
- new net GND: J19.1 (Pin_1)
- new net SCK: J19.5 (Pin_5)
Changed lines of the file:
@@
 $Descr A4 11693 8268
 encoding utf-8
-Sheet 1 6
+Sheet 5 6
 Title ""
 Date ""
@@
 Comment4 ""
 $EndDescr
+$Comp
+L Conn_01x05_Female J19
+U 1 1 5ACF0297
+P 4850 3600
+F 0 "J19" H 4850 3900 50  0000 C CNN
+F 1 "MAX6675" H 4850 3300 50  0000 C CNN
+F 2 "Socket_Strips:Socket_Strip_Straight_1x05_Pitch2.54mm" H 4850 3600 50  0001 C CNN
+F 3 "" H 4850 3600 50  0001 C CNN
+	1    4850 3600
+	-1   0    0    1
+$EndComp
+$Comp
+L GND #PWR011
+U 1 1 5ACF0334
+P 5450 3800
+F 0 "#PWR011" H 5450 3550 50  0001 C CNN
+F 1 "GND" H 5450 3650 50  0000 C CNN
+F 2 "" H 5450 3800 50  0001 C CNN
+F 3 "" H 5450 3800 50  0001 C CNN
+	1    5450 3800
+	0    -1   -1   0
+$EndComp
+$Comp
+L +5V #PWR012
+U 1 1 5ACF0357
+P 5850 3700
+F 0 "#PWR012" H 5850 3550 50  0001 C CNN
+F 1 "+5V" H 5850 3840 50  0000 C CNN
+F 2 "" H 5850 3700 50  0001 C CNN
+F 3 "" H 5850 3700 50  0001 C CNN
+	1    5850 3700
+	0    1    1    0
+$EndComp
+Text HLabel 5600 3600 2    60   Input ~ 0
+90
+Text HLabel 5600 3500 2    60   Input ~ 0
+CS
+Text HLabel 5600 3400 2    60   Input ~ 0
+SCK
+Wire Wire Line
+	5450 3800 5050 3800
+Wire Wire Line
+	5050 3700 5850 3700
+Wire Wire Line
+	5600 3600 5050 3600
+Wire Wire Line
+	5050 3500 5600 3500
+Wire Wire Line
+	5050 3400 5600 3400
 $EndSCHEMATC
