File: stepperControl.sch (KiCad schematic (older format))
At the start: 18 parts, among them J1 pulX, J2 dirX, J3 enaX, J4 pulY, J5 dirY, J6 enaY, J7 pulZ, J8 dirZ, J9 enaZ, Q1 Q_NPN_CBE, Q2 Q_NPN_CBE, Q3 Q_NPN_CBE, Q4 Q_NPN_CBE, Q5 Q_NPN_CBE, Q6 Q_NPN_CBE, Q7 Q_NPN_CBE, Q8 Q_NPN_CBE, Q9 Q_NPN_CBE

Commit message: Add files via upload
Parts:
- added J16: pulX0, Connectors_Terminal_Blocks:TerminalBlock_Altech_AK300-2_P5.00mm, symbol Screw_Terminal_01x02
- added J17: dirX0, Connectors_Terminal_Blocks:TerminalBlock_Altech_AK300-2_P5.00mm, symbol Screw_Terminal_01x02
- added J18: enaX0, Connectors_Terminal_Blocks:TerminalBlock_Altech_AK300-2_P5.00mm, symbol Screw_Terminal_01x02
- added Q14, Q15, Q16: Q_NPN_CBE, TO_SOT_Packages_THT:TO-92_Inline_Narrow_Oval, symbol Q_NPN_CBE
- added R10, R11, R12, R13, R14, R15, R16, R17, R18, R7, R8, R9: R, Resistors_THT:R_Axial_DIN0207_L6.3mm_D2.5mm_P10.16mm_Horizontal, symbol R
- J1: value pulX -> pulX1
- J2: value dirX -> dirX1
- J3: value enaX -> enaX1
Connections:
- net +5V: now also J16.1 (Pin_1), J17.1 (Pin_1), J18.1 (Pin_1)
- net GND: now also Q14.3 (E), Q15.3 (E), Q16.3 (E)
- net at J1.2 (Pin_2): now also R10.1; no longer Q1.1 (C)
- net at J2.2 (Pin_2): now also R11.1; no longer Q2.1 (C)
- net at J3.2 (Pin_2): now also R12.1; no longer Q3.1 (C)
- net at J4.2 (Pin_2): now also R13.1; no longer Q4.1 (C)
- net at J5.2 (Pin_2): now also R14.1; no longer Q5.1 (C)
- net at J6.2 (Pin_2): now also R15.1; no longer Q6.1 (C)
- net at J7.2 (Pin_2): now also R16.1; no longer Q7.1 (C)
- net at J8.2 (Pin_2): now also R17.1; no longer Q8.1 (C)
- net at J9.2 (Pin_2): now also R18.1; no longer Q9.1 (C)
- net PulX renamed PulX1
- net dirX renamed dirX1
- net enaX renamed enaX1
- new net: Q1.1 (C), R10.2
- new net: Q2.1 (C), R11.2
- new net: Q3.1 (C), R12.2
- new net: Q4.1 (C), R13.2
- new net: Q5.1 (C), R14.2
- new net: Q6.1 (C), R15.2
- new net: Q7.1 (C), R16.2
- new net: Q8.1 (C), R17.2
- new net: Q9.1 (C), R18.2
- new net: J16.2 (Pin_2), R7.1
- new net: J17.2 (Pin_2), R8.1
- new net: J18.2 (Pin_2), R9.1
- new net: Q14.1 (C), R7.2
- new net: Q15.1 (C), R8.2
- new net: Q16.1 (C), R9.2
- new net PulX0: Q14.2 (B)
- new net dirX0: Q15.2 (B)
- new net enaX0: Q16.2 (B)
Other:
- moved on the sheet: J1, J2, J3, J4, J5, J6, J7, J8, J9, Q1, Q2, Q3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

Commit message: Add files via upload
Parts:
- added J22: XMin, symbol Screw_Terminal_01x02
- added J23: XMax, symbol Screw_Terminal_01x02
- added J25: YMin, symbol Screw_Terminal_01x02
- added J26: YMax, symbol Screw_Terminal_01x02
- added J27: ZMin, symbol Screw_Terminal_01x02
- added J32: ZMax, symbol Screw_Terminal_01x02
- added Q17, Q18, Q19, Q20, Q21, Q22: Q_NPN_CBE, symbol Q_NPN_CBE
- added R19, R20, R21, R22, R23, R24: R, symbol R
Connections:
- net +5V: now also J22.1 (Pin_1), J23.1 (Pin_1), J25.1 (Pin_1), J26.1 (Pin_1), J27.1 (Pin_1), J32.1 (Pin_1)
- net GND: now also Q17.3 (E), Q18.3 (E), Q19.3 (E), Q20.3 (E), Q21.3 (E), Q22.3 (E)
- net at Q3.1 (C), R12.2: now also Q15.1 (C), R8.2, Q17.1 (C), Q18.1 (C)
- net at Q6.1 (C), R15.2: now also Q19.1 (C), Q20.1 (C)
- net at Q9.1 (C), R18.2: now also Q21.1 (C), Q22.1 (C)
- new net: J23.2 (Pin_2), Q18.2 (B), R20.1
- new net: J22.2 (Pin_2), Q17.2 (B), R19.1
- new net: J26.2 (Pin_2), Q20.2 (B), R22.1
- new net: J25.2 (Pin_2), Q19.2 (B), R21.1
- new net: J32.2 (Pin_2), Q22.2 (B), R24.1
- new net: J27.2 (Pin_2), Q21.2 (B), R23.1
- new net XMax: R20.2
- new net XMin: R19.2
- new net YMax: R22.2
- new net YMin: R21.2
- new net ZMax: R24.2
- new net ZMin: R23.2
Other:
- moved on the sheet: J1, J16, J17, J18, J2, J3, J4, J5, J6, J7, J8, J9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
